File: pcb/baja_daq.kicad_pcb (KiCad board)
At the start: 4 copper layers, 65 x 65 mm, 57 parts, among them J1 Micro_SD_Card, J3 Conn_01x03, J4 Conn_01x03, J7 Conn_01x02, U1 STM32F405RGTx, U2 TJA1051T, U4 L7805, U5 AMS1117-3.3, Y1 8MHz

Commit message: updated firmware
Parts:
- moved C1 15.1 mm to (104.5, 107.0)
- moved Y1 14.1 mm to (101.2, 108.8), turned to -90 degrees
- moved C2 11.0 mm to (104.5, 110.5), turned to -90 degrees
- moved CAN 8.25 mm to (98.0, 118.2)
- moved C13 0.90 mm to (106.2, 111.5), turned to -90 degrees
- moved R7 0.81 mm to (93.1, 104.5)
- moved C7 0.53 mm to (107.2, 106.0)
Routing:
- net N$4: track 23.0 -> 9.29 mm
- net N$5: track 19.6 -> 7.80 mm
- net CAN_P: track 12.3 -> 20.3 mm
- net CAN_N: track 11.3 -> 19.3 mm
- net GND: track 48.6 -> 47.0 mm, vias 73 -> 81
- net N$2: track 36.2 -> 37.5 mm
- net +3V3_DIG: track 48.9 -> 47.7 mm
